File: kicad/scamp-plus/_restore_backup_2026-09-13T19-42-04-211/scamp++.kicad_sch (KiCad schematic)
At the start: 66 parts, among them J1 Conn_02x25_Top_Bottom, J2 Conn_01x03_Pin, J3 Conn_01x02_Pin, J4 DIN41612_03x32_C_Split, U1 74ACT377, U10 74ACT32, U11 74ACT02, U12 74ACT377, U2 74ACT377, U3 74ACT244, U4 74ACT244, U5 74ACT377, U6 74ACT377, U7 74ACT32, U8 74ACT32, U9 74ACT32

Commit message: add jnz. support for reversing byte order due to limited t-cycles
Other:
- note removed: "NOTE TO BEN! This might not be right. Check logisim for z_new. Had to and two nor's"
