File: kicad/scamp32-memory/scamp32-memory.kicad_pcb (KiCad board)
At the start: 4 copper layers, 100 x 160 mm, 10 parts, among them J1 DIN41612_C_3x32, J2 PWR_5V, SW1 SW_SPST

Commit message: template and memory board
Parts:
- added C1: 100nF, Capacitor_SMD:C_0603_1608Metric, F.Cu at (57.5, 59.0)
- added C10: 100nF, Capacitor_SMD:C_0603_1608Metric, F.Cu at (89.2, 41.2)
- added C11: 100nF, Capacitor_SMD:C_0603_1608Metric, F.Cu at (99.0, 41.2)
- added C12: 100nF, Capacitor_SMD:C_0603_1608Metric, F.Cu at (108.8, 41.2)
- added C13: 100nF, Capacitor_SMD:C_0603_1608Metric, F.Cu at (118.5, 41.2)
- added C14: 100nF, Capacitor_SMD:C_0603_1608Metric, F.Cu at (128.2, 41.2)
- added C15: 100nF, Capacitor_SMD:C_0603_1608Metric, F.Cu at (137.8, 41.2)
- added C16: 100nF, Capacitor_SMD:C_0603_1608Metric, F.Cu at (69.5, 66.0)
- added C17: 100nF, Capacitor_SMD:C_0603_1608Metric, F.Cu at (79.2, 65.9)
- added C18: C51, Capacitor_SMD:C_0603_1608Metric, F.Cu at (89.0, 65.9)
- added C19: 100nF, Capacitor_SMD:C_0603_1608Metric, F.Cu at (98.8, 65.9)
- added C2: 100nF, Capacitor_SMD:C_0603_1608Metric, F.Cu at (57.5, 50.0)
- added C20: 100nF, Capacitor_SMD:C_0603_1608Metric, F.Cu at (108.5, 66.0)
- added C21: 100nF, Capacitor_SMD:C_0603_1608Metric, F.Cu at (118.2, 66.0)
- added C22: 100nF, Capacitor_SMD:C_0603_1608Metric, F.Cu at (128.0, 66.0)
- added C23: 100nF, Capacitor_SMD:C_0603_1608Metric, F.Cu at (137.5, 66.0)
- added C24: 100nF, Capacitor_SMD:C_0603_1608Metric, F.Cu at (69.8, 54.0)
- added C25: 100nF, Capacitor_SMD:C_0603_1608Metric, F.Cu at (79.5, 54.0)
- added C26: C51, Capacitor_SMD:C_0603_1608Metric, F.Cu at (89.0, 54.0)
- added C27: 100nF, Capacitor_SMD:C_0603_1608Metric, F.Cu at (99.0, 54.0)
- added C28: 100nF, Capacitor_SMD:C_0603_1608Metric, F.Cu at (108.5, 54.0)
- added C29: 100nF, Capacitor_SMD:C_0603_1608Metric, F.Cu at (118.2, 54.0)
- added C3: 100nF, Capacitor_SMD:C_0603_1608Metric, F.Cu at (118.0, 144.0)
- added C30: 100nF, Capacitor_SMD:C_0603_1608Metric, F.Cu at (128.0, 54.0)
- added C31: 100nF, Capacitor_SMD:C_0603_1608Metric, F.Cu at (137.8, 54.0)
- added C32: 100nF, Capacitor_SMD:C_0603_1608Metric, F.Cu at (94.8, 78.8)
- added C33: 100nF, Capacitor_SMD:C_0603_1608Metric, F.Cu at (84.5, 78.8)
- added C34: 100nF, Capacitor_SMD:C_0603_1608Metric, F.Cu at (73.0, 79.0)
- added C35: 100nF, Capacitor_SMD:C_0603_1608Metric, F.Cu at (62.0, 79.0)
- added C36: 100nF, Capacitor_SMD:C_0603_1608Metric, F.Cu at (94.8, 92.1)
- added C37: 100nF, Capacitor_SMD:C_0603_1608Metric, F.Cu at (84.3, 92.1)
- added C38: 100nF, Capacitor_SMD:C_0603_1608Metric, F.Cu at (72.8, 92.1)
- added C39: 100nF, Capacitor_SMD:C_0603_1608Metric, F.Cu at (62.4, 92.1)
- added C4: 100nF, Capacitor_SMD:C_0603_1608Metric, F.Cu at (134.8, 131.8)
- added C40: 100nF, Capacitor_SMD:C_0603_1608Metric, F.Cu at (127.0, 79.0)
- added C41: 100nF, Capacitor_SMD:C_0603_1608Metric, F.Cu at (138.0, 79.0)
- added C42: 100nF, Capacitor_SMD:C_0603_1608Metric, F.Cu at (116.5, 79.0)
- added C43: 100nF, Capacitor_SMD:C_0603_1608Metric, F.Cu at (105.2, 79.0)
- added C44: 100nF, Capacitor_SMD:C_0603_1608Metric, F.Cu at (126.8, 92.1)
- added C45: 100nF, Capacitor_SMD:C_0603_1608Metric, F.Cu at (138.1, 92.1)
- added C46: 100nF, Capacitor_SMD:C_0603_1608Metric, F.Cu at (116.1, 92.1)
- added C47: 100nF, Capacitor_SMD:C_0603_1608Metric, F.Cu at (105.1, 92.1)
- added C48: 100nF, Capacitor_SMD:C_0603_1608Metric, F.Cu at (79.5, 41.2)
- added C5: 100nF, Capacitor_SMD:C_0603_1608Metric, F.Cu at (94.2, 131.5)
- added C6: 100nF, Capacitor_SMD:C_0603_1608Metric, F.Cu at (134.8, 159.7)
- added C7: 100nF, Capacitor_SMD:C_0603_1608Metric, F.Cu at (94.2, 159.2)
- added C8: 100nF, Capacitor_SMD:C_0603_1608Metric, F.Cu at (69.8, 41.2)
- added J1: Conn_02x20_Counter_Clockwise, Connector_IDC:IDC-Header_2x20_P2.54mm_Horizontal, F.Cu at (115.6, 172.5)
- added JP1: SolderJumper_3_Open, Jumper:SolderJumper-3_P1.3mm_Open_RoundedPad1.0x1.5mm_NumberLabels, F.Cu at (118.7, 167.5)
- added JP10: SolderJumper_3_Open, Jumper:SolderJumper-3_P1.3mm_Open_RoundedPad1.0x1.5mm_NumberLabels, F.Cu at (64.5, 163.8)
- added JP11: SolderJumper_3_Open, Jumper:SolderJumper-3_P1.3mm_Open_RoundedPad1.0x1.5mm_NumberLabels, F.Cu at (71.1, 167.6)
- added JP12: SolderJumper_3_Open, Jumper:SolderJumper-3_P1.3mm_Open_RoundedPad1.0x1.5mm_NumberLabels, F.Cu at (71.3, 163.6)
- added JP13: SolderJumper_3_Open, Jumper:SolderJumper-3_P1.3mm_Open_RoundedPad1.0x1.5mm_NumberLabels, F.Cu at (78.0, 167.5)
- added JP14: SolderJumper_3_Open, Jumper:SolderJumper-3_P1.3mm_Open_RoundedPad1.0x1.5mm_NumberLabels, F.Cu at (77.9, 163.5)
- added JP15: SolderJumper_3_Open, Jumper:SolderJumper-3_P1.3mm_Open_RoundedPad1.0x1.5mm_NumberLabels, F.Cu at (84.7, 167.4)
- added JP16: SolderJumper_3_Open, Jumper:SolderJumper-3_P1.3mm_Open_RoundedPad1.0x1.5mm_NumberLabels, F.Cu at (84.6, 163.6)
- added JP17: SolderJumper_3_Open, Jumper:SolderJumper-3_P1.3mm_Open_RoundedPad1.0x1.5mm_NumberLabels, F.Cu at (91.6, 167.4)
- added JP18: SolderJumper_3_Open, Jumper:SolderJumper-3_P1.3mm_Open_RoundedPad1.0x1.5mm_NumberLabels, F.Cu at (91.6, 163.6)
- added JP19: SolderJumper_3_Open, Jumper:SolderJumper-3_P1.3mm_Open_RoundedPad1.0x1.5mm_NumberLabels, F.Cu at (61.5, 73.8)
- added JP2: SolderJumper_3_Open, Jumper:SolderJumper-3_P1.3mm_Open_RoundedPad1.0x1.5mm_NumberLabels, F.Cu at (118.8, 163.5)
- added JP20: SolderJumper_3_Open, Jumper:SolderJumper-3_P1.3mm_Open_RoundedPad1.0x1.5mm_NumberLabels, F.Cu at (61.5, 69.5)
- added JP3: SolderJumper_3_Open, Jumper:SolderJumper-3_P1.3mm_Open_RoundedPad1.0x1.5mm_NumberLabels, F.Cu at (111.9, 167.5)
- added JP4: SolderJumper_3_Open, Jumper:SolderJumper-3_P1.3mm_Open_RoundedPad1.0x1.5mm_NumberLabels, F.Cu at (112.0, 163.5)
- added JP5: SolderJumper_3_Open, Jumper:SolderJumper-3_P1.3mm_Open_RoundedPad1.0x1.5mm_NumberLabels, F.Cu at (105.2, 167.5)
- added JP6: SolderJumper_3_Open, Jumper:SolderJumper-3_P1.3mm_Open_RoundedPad1.0x1.5mm_NumberLabels, F.Cu at (105.2, 163.5)
- added JP7: SolderJumper_3_Open, Jumper:SolderJumper-3_P1.3mm_Open_RoundedPad1.0x1.5mm_NumberLabels, F.Cu at (98.4, 167.5)
- added JP8: SolderJumper_3_Open, Jumper:SolderJumper-3_P1.3mm_Open_RoundedPad1.0x1.5mm_NumberLabels, F.Cu at (98.4, 163.5)
- added JP9: SolderJumper_3_Open, Jumper:SolderJumper-3_P1.3mm_Open_RoundedPad1.0x1.5mm_NumberLabels, F.Cu at (64.4, 167.5)
- added U1: 74ACT08, Package_SO:TSSOP-14_4.4x5mm_P0.65mm, F.Cu at (61.5, 62.2)
- added U10: 74ACT283, Package_SO:TSSOP-16_4.4x5mm_P0.65mm, F.Cu at (91.4, 47.2)
- added U11: 74ACT283, Package_SO:TSSOP-16_4.4x5mm_P0.65mm, F.Cu at (101.1, 47.2)
- added U12: 74ACT283, Package_SO:TSSOP-16_4.4x5mm_P0.65mm, F.Cu at (110.9, 47.2)
- added U13: 74ACT283, Package_SO:TSSOP-16_4.4x5mm_P0.65mm, F.Cu at (120.6, 47.2)
- added U14: 74ACT283, Package_SO:TSSOP-16_4.4x5mm_P0.65mm, F.Cu at (130.3, 47.2)
- added U15: 74ACT283, Package_SO:TSSOP-16_4.4x5mm_P0.65mm, F.Cu at (140.0, 47.2)
- added U16: 74ACT157, Package_SO:TSSOP-16_4.4x5mm_P0.65mm, F.Cu at (72.0, 71.9)
- added U17: 74ACT157, Package_SO:TSSOP-16_4.4x5mm_P0.65mm, F.Cu at (81.7, 71.9)
- added U18: 74ACT157, Package_SO:TSSOP-16_4.4x5mm_P0.65mm, F.Cu at (91.4, 71.9)
- added U19: 74ACT157, Package_SO:TSSOP-16_4.4x5mm_P0.65mm, F.Cu at (101.1, 71.9)
- added U2: 74ACT32, Package_SO:TSSOP-14_4.4x5mm_P0.65mm, F.Cu at (61.5, 52.5)
- added U20: 74ACT157, Package_SO:TSSOP-16_4.4x5mm_P0.65mm, F.Cu at (110.8, 71.9)
- added U21: 74ACT157, Package_SO:TSSOP-16_4.4x5mm_P0.65mm, F.Cu at (120.5, 71.9)
- added U22: 74ACT157, Package_SO:TSSOP-16_4.4x5mm_P0.65mm, F.Cu at (130.3, 71.9)
- added U23: 74ACT157, Package_SO:TSSOP-16_4.4x5mm_P0.65mm, F.Cu at (140.0, 71.9)
- added U24: 74ACT157, Package_SO:TSSOP-16_4.4x5mm_P0.65mm, F.Cu at (72.0, 59.8)
- added U25: 74ACT157, Package_SO:TSSOP-16_4.4x5mm_P0.65mm, F.Cu at (81.7, 59.8)
- added U26: 74ACT157, Package_SO:TSSOP-16_4.4x5mm_P0.65mm, F.Cu at (91.4, 59.8)
- added U27: 74ACT157, Package_SO:TSSOP-16_4.4x5mm_P0.65mm, F.Cu at (101.1, 59.8)
- added U28: 74ACT157, Package_SO:TSSOP-16_4.4x5mm_P0.65mm, F.Cu at (110.8, 59.8)
- added U29: 74ACT157, Package_SO:TSSOP-16_4.4x5mm_P0.65mm, F.Cu at (120.5, 59.8)
- added U3: 74ACT02, Package_SO:TSSOP-14_4.4x5mm_P0.65mm, F.Cu at (120.0, 150.0)
- added U30: 74ACT157, Package_SO:TSSOP-16_4.4x5mm_P0.65mm, F.Cu at (130.3, 59.8)
- added U31: 74ACT157, Package_SO:TSSOP-16_4.4x5mm_P0.65mm, F.Cu at (140.0, 59.8)
- added U32: 74ACT244, Package_SO:Texas_PW0020A_TSSOP-20_4.4x6.5mm_P0.65mm, F.Cu at (97.7, 85.2)
- added U33: 74ACT244, Package_SO:Texas_PW0020A_TSSOP-20_4.4x6.5mm_P0.65mm, F.Cu at (87.5, 85.2)
- added U34: 74ACT244, Package_SO:Texas_PW0020A_TSSOP-20_4.4x6.5mm_P0.65mm, F.Cu at (76.1, 85.2)
- added U35: 74ACT244, Package_SO:Texas_PW0020A_TSSOP-20_4.4x6.5mm_P0.65mm, F.Cu at (65.0, 85.2)
- added U36: 74ACT244, Package_SO:Texas_PW0020A_TSSOP-20_4.4x6.5mm_P0.65mm, F.Cu at (97.8, 98.2)
- added U37: 74ACT244, Package_SO:Texas_PW0020A_TSSOP-20_4.4x6.5mm_P0.65mm, F.Cu at (87.3, 98.2)
- added U38: 74ACT244, Package_SO:Texas_PW0020A_TSSOP-20_4.4x6.5mm_P0.65mm, F.Cu at (75.9, 98.2)
- added U39: 74ACT244, Package_SO:Texas_PW0020A_TSSOP-20_4.4x6.5mm_P0.65mm, F.Cu at (65.4, 98.2)
- added U4: AS6C4008-55TIN, Package_SO:TSOP-I-32_18.4x8mm_P0.5mm, F.Cu at (135.0, 118.0)
- added U40: 74ACT244, Package_SO:Texas_PW0020A_TSSOP-20_4.4x6.5mm_P0.65mm, F.Cu at (130.0, 85.2)
- added U41: 74ACT244, Package_SO:Texas_PW0020A_TSSOP-20_4.4x6.5mm_P0.65mm, F.Cu at (141.0, 85.2)
- added U42: 74ACT244, Package_SO:Texas_PW0020A_TSSOP-20_4.4x6.5mm_P0.65mm, F.Cu at (119.5, 85.2)
- added U43: 74ACT244, Package_SO:Texas_PW0020A_TSSOP-20_4.4x6.5mm_P0.65mm, F.Cu at (108.2, 85.2)
- added U44: 74ACT244, Package_SO:Texas_PW0020A_TSSOP-20_4.4x6.5mm_P0.65mm, F.Cu at (129.8, 98.2)
- added U45: 74ACT244, Package_SO:Texas_PW0020A_TSSOP-20_4.4x6.5mm_P0.65mm, F.Cu at (141.0, 98.2)
- added U46: 74ACT244, Package_SO:Texas_PW0020A_TSSOP-20_4.4x6.5mm_P0.65mm, F.Cu at (119.0, 98.2)
- added U47: 74ACT244, Package_SO:Texas_PW0020A_TSSOP-20_4.4x6.5mm_P0.65mm, F.Cu at (108.0, 98.2)
- added U5: FM1608B-SG, Socket:DIP_Socket-28_W11.9mm_W12.7mm_W15.24mm_W17.78mm_W18.5mm_3M_228-1277-00-0602J, F.Cu at (96.0, 110.0)
- added U6: AS6C4008-55TIN, Package_SO:TSOP-I-32_18.4x8mm_P0.5mm, F.Cu at (135.0, 146.0)
- added U7: FM1608B-SG, Socket:DIP_Socket-28_W11.9mm_W12.7mm_W15.24mm_W17.78mm_W18.5mm_3M_228-1277-00-0602J, F.Cu at (96.0, 138.0)
- added U8: 74ACT283, Package_SO:TSSOP-16_4.4x5mm_P0.65mm, F.Cu at (72.0, 47.2)
- added U9: 74ACT283, Package_SO:TSSOP-16_4.4x5mm_P0.65mm, F.Cu at (81.7, 47.2)
- moved LED1 34.1 mm to (148.0, 175.0), turned to 0 degrees
- moved R1 33.5 mm to (148.1, 170.0)
- moved SW1 2.50 mm to (124.9, 184.0)
- moved C49 2.47 mm to (126.0, 177.0)
- moved J3 1.00 mm to (135.9, 181.0)
- renumbered C1 to C49, J1 to J2, J2 to J3
Connections:
- net AI renamed ~{AI}
- net DI renamed ~{DI}
- net DO renamed ~{DO}
- net EO renamed ~{EO}
- net II renamed ~{II}
- net IVI renamed ~{IVI}
- net IVO renamed ~{IVO}
- net MB renamed ~{MB}
- net MH renamed ~{MH}
- net MI renamed ~{MI}
- net MO renamed ~{MO}
- net MW renamed ~{MW}
- net PO renamed ~{PO}
- net PP1 renamed ~{PP1}
- net PP2 renamed ~{PP2}
- net PP4 renamed ~{PP4}
- net SI renamed ~{SI}
- net SO renamed ~{SO}
- net XI renamed ~{XI}
- net YI renamed ~{YI}
Routing:
- net GND: track 0.00 -> 477.9 mm, vias 0 -> 55
- net VCC: track 2.17 -> 351.4 mm, vias 1 -> 51
- net /D14: track 0.00 -> 301.0 mm, vias 0 -> 10
- net /D17: track 0.00 -> 299.7 mm, vias 0 -> 10
- net /D15: track 0.00 -> 299.0 mm, vias 0 -> 10
- net /D16: track 0.00 -> 296.7 mm, vias 0 -> 10
- net /D05: track 0.00 -> 283.8 mm, vias 0 -> 9
- net /D07: track 0.00 -> 278.2 mm, vias 0 -> 9
- net /D06: track 0.00 -> 277.9 mm, vias 0 -> 9
- net /samp32-memory-mux/A_SEL12: track 0.00 -> 266.5 mm, vias 0 -> 6
- net /samp32-memory-mux/A_SEL8: track 0.00 -> 249.9 mm, vias 0 -> 6
- net /D04: track 0.00 -> 246.6 mm, vias 0 -> 11
- net /samp32-memory-mux/A_SEL11: track 0.00 -> 240.1 mm, vias 0 -> 5
- net /samp32-memory-mux/A_SEL9: track 0.00 -> 238.5 mm, vias 0 -> 6
- net /samp32-memory-mux/A_SEL10: track 0.00 -> 238.1 mm, vias 0 -> 5
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Other:
- board text added: "CHIP SELECT"
