File: kicad/scamp32-memory/scamp32-memory.kicad_sch (KiCad schematic)
At the start: 6 parts, among them J1 DIN41612_C_3x32, J2 PWR_5V, SW1 SW_SPST

Commit message: template and memory board
Parts:
- added C1, C2, C3, C4, C5, C6, C7: 100nF, Capacitor_SMD:C_0603_1608Metric, symbol Device:C
- added J1: Conn_02x20_Counter_Clockwise, Connector_IDC:IDC-Header_2x20_P2.54mm_Horizontal, symbol Connector_Generic:Conn_02x20_Counter_Clockwise
- added JP1, JP10, JP11, JP12, JP13, JP14, JP15, JP16, JP17, JP18, JP19, JP2, JP20, JP3, JP4, JP5, JP6, JP7, JP8, JP9: SolderJumper_3_Open, Jumper:SolderJumper-3_P1.3mm_Open_RoundedPad1.0x1.5mm_NumberLabels, symbol Jumper:SolderJumper_3_Open
- added U1: 74ACT08, Package_SO:TSSOP-14_4.4x5mm_P0.65mm, symbol scamp_act:74ACT08
- added U2: 74ACT32, Package_SO:SOIC-14_3.9x8.7mm_P1.27mm, symbol scamp_act:74ACT32
- added U3: 74ACT02, Package_SO:TSSOP-14_4.4x5mm_P0.65mm, symbol scamp_act:74ACT02
- added U4, U6: AS6C4008-55TIN, Package_SO:TSOP-I-32_18.4x8mm_P0.5mm, symbol scamp_memory:AS6C4008-55TIN
- added U5, U7: FM1608B-SG, Socket:DIP_Socket-28_W11.9mm_W12.7mm_W15.24mm_W17.78mm_W18.5mm_3M_228-1277-00-0602J, symbol scamp_memory:FM1608B-SG
- renumbered C1 to C49, J1 to J2, J2 to J3
Connections:
- net A0: now also U1.1, U2.1
- net A1: now also JP19.3 (B), U1.2, U2.2
- net GND: now also C1.2, C2.2, C3.2, C4.2, C5.2, C6.2, C7.2, JP19.1 (A), U1.7 (GND), U2.7 (GND), U3.7 (GND), U4.24 (VSS), U5.14 (VSS), U5.20 (~{CE}), U6.24 (VSS), U7.14 (VSS), U7.20 (~{CE})
- net VCC: now also C1.1, C2.1, C3.1, C4.1, C5.1, C6.1, C7.1, U1.14 (VCC), U2.14 (VCC), U3.14 (VCC), U4.8 (VCC), U5.27 (~{WE}), U5.28 (VDD), U6.8 (VCC), U7.27 (~{WE}), U7.28 (VDD)
- net AI renamed ~{AI}
- net DI renamed ~{DI}
- net DO renamed ~{DO}
- net EO renamed ~{EO}
- net II renamed ~{II}
- net IVI renamed ~{IVI}
- net IVO renamed ~{IVO}
- net MB renamed ~{MB}
- net MH renamed ~{MH}
- net MI renamed ~{MI}
- net MO renamed ~{MO}
- net MW renamed ~{MW}
- net PO renamed ~{PO}
- net PP1 renamed ~{PP1}
- net PP2 renamed ~{PP2}
- net PP4 renamed ~{PP4}
- net SI renamed ~{SI}
- net SO renamed ~{SO}
- net XI renamed ~{XI}
- net YI renamed ~{YI}
- new net: U3.13, U6.30 (CE#)
- new net: JP20.3 (B), U2.3
- new net: U3.4, U7.22 (~{OE})
- new net: U3.1, U5.22 (~{OE})
- new net: JP20.1 (A), U1.3
- new net: U3.10, U4.30 (CE#)
- new net A_SEL0: U4.20 (A0), U5.10 (A0), U6.20 (A0), U7.10 (A0)
- new net A_SEL1: U4.19 (A1), U5.9 (A1), U6.19 (A1), U7.9 (A1)
- new net A_SEL10: U4.31 (A10), U5.21 (A10), U6.31 (A10), U7.21 (A10)
- new net A_SEL11: U4.1 (A11), U5.23 (A11), U6.1 (A11), U7.23 (A11)
- new net A_SEL12: U4.12 (A12), U5.2 (A12), U6.12 (A12), U7.2 (A12)
- new net A_SEL13: U4.4 (A13), U6.4 (A13)
- new net A_SEL14: U4.11 (A14), U6.11 (A14)
- new net A_SEL15: U4.7 (A15), U6.7 (A15)
- new net A_SEL16: U4.10 (A16), U6.10 (A16)
- new net A_SEL17: U4.6 (A17), U6.6 (A17)
- new net A_SEL18: U4.9 (A18), U6.9 (A18)
- new net A_SEL2: U4.18 (A2), U5.8 (A2), U6.18 (A2), U7.8 (A2)
- new net A_SEL3: U4.17 (A3), U5.7 (A3), U6.17 (A3), U7.7 (A3)
- new net A_SEL4: U4.16 (A4), U5.6 (A4), U6.16 (A4), U7.6 (A4)
- new net A_SEL5: U4.14 (A5), U5.5 (A5), U6.14 (A5), U7.5 (A5)
- new net A_SEL6: U4.15 (A6), U5.4 (A6), U6.15 (A6), U7.4 (A6)
- new net A_SEL7: U4.13 (A7), U5.3 (A7), U6.13 (A7), U7.3 (A7)
- new net A_SEL8: U4.3 (A8), U5.25 (A8), U6.3 (A8), U7.25 (A8)
- new net A_SEL9: U4.2 (A9), U5.24 (A9), U6.2 (A9), U7.24 (A9)
- new net D00: U4.21 (DQ0), U5.11 (DQ0)
- new net D01: U4.22 (DQ1), U5.12 (DQ1)
- new net D02: U4.23 (DQ2), U5.13 (DQ2)
- new net D03: U4.25 (DQ3), U5.15 (DQ3)
- new net D04: U4.26 (DQ4), U5.16 (DQ4)
- new net D05: U4.27 (DQ5), U5.17 (DQ5)
- new net D06: U4.28 (DQ6), U5.18 (DQ6)
- new net D07: U4.29 (DQ7), U5.19 (DQ7)
- new net D10: U6.21 (DQ0), U7.11 (DQ0)
- new net D11: U6.22 (DQ1), U7.12 (DQ1)
- new net D12: U6.23 (DQ2), U7.13 (DQ2)
- new net D13: U6.25 (DQ3), U7.15 (DQ3)
- new net D14: U6.26 (DQ4), U7.16 (DQ4)
- new net D15: U6.27 (DQ5), U7.17 (DQ5)
- new net D16: U6.28 (DQ6), U7.18 (DQ6)
- new net D17: U6.29 (DQ7), U7.19 (DQ7)
- new net samp32-memory-mux/S: JP20.2 (C)
- new net samp32-memory-mux1/S: JP19.2 (C)
- new net ~{CHIP_0}: J1.17 (Pin_17), JP17.3 (B)
- new net ~{CHIP_1}: J1.18 (Pin_18), JP18.3 (B)
- new net ~{CHIP_2}: J1.24 (Pin_24), JP17.1 (A)
- new net ~{CHIP_3}: J1.23 (Pin_23), JP18.1 (A)
- new net ~{LOAD_CLK}: J1.20 (Pin_20), U4.5 (WE#), U6.5 (WE#)
- new net ~{MI0_0}: J1.1 (Pin_1), JP1.3 (B)
- new net ~{MI0_1}: J1.2 (Pin_2), JP2.3 (B)
- new net ~{MI0_2}: J1.3 (Pin_3), JP3.3 (B)
- new net ~{MI0_3}: J1.4 (Pin_4), JP4.3 (B)
- new net ~{MI1_0}: J1.40 (Pin_40), JP9.3 (B)
- new net ~{MI1_1}: J1.39 (Pin_39), JP10.3 (B)
- new net ~{MI1_2}: J1.38 (Pin_38), JP11.3 (B)
- new net ~{MI1_3}: J1.37 (Pin_37), JP12.3 (B)
- new net ~{MI2_0}: J1.5 (Pin_5), JP1.1 (A)
- new net ~{MI2_1}: J1.6 (Pin_6), JP2.1 (A)
- new net ~{MI2_2}: J1.7 (Pin_7), JP3.1 (A)
- new net ~{MI2_3}: J1.8 (Pin_8), JP4.1 (A)
- new net ~{MI3_0}: J1.36 (Pin_36), JP9.1 (A)
- new net ~{MI3_1}: J1.35 (Pin_35), JP10.1 (A)
- new net ~{MI3_2}: J1.34 (Pin_34), JP11.1 (A)
- new net ~{MI3_3}: J1.33 (Pin_33), JP12.1 (A)
- new net ~{MI_S0_0}: JP1.2 (C)
- new net ~{MI_S0_1}: JP2.2 (C)
- new net ~{MI_S0_2}: JP3.2 (C)
- new net ~{MI_S0_3}: JP4.2 (C)
- new net ~{MI_S1_0}: JP9.2 (C)
- new net ~{MI_S1_1}: JP10.2 (C)
- new net ~{MI_S1_2}: JP11.2 (C)
- new net ~{MI_S1_3}: JP12.2 (C)
- new net ~{MO0_0}: J1.9 (Pin_9), JP5.3 (B)
- new net ~{MO0_1}: J1.10 (Pin_10), JP6.3 (B)
- new net ~{MO0_2}: J1.11 (Pin_11), JP7.3 (B)
- new net ~{MO0_3}: J1.12 (Pin_12), JP8.3 (B)
- new net ~{MO1_0}: J1.32 (Pin_32), JP13.3 (B)
- new net ~{MO1_1}: J1.31 (Pin_31), JP14.3 (B)
- new net ~{MO1_2}: J1.30 (Pin_30), JP15.3 (B)
- new net ~{MO1_3}: J1.29 (Pin_29), JP16.3 (B)
- new net ~{MO2_0}: J1.13 (Pin_13), JP5.1 (A)
- new net ~{MO2_1}: J1.14 (Pin_14), JP6.1 (A)
- new net ~{MO2_2}: J1.15 (Pin_15), JP7.1 (A)
- new net ~{MO2_3}: J1.16 (Pin_16), JP8.1 (A)
- new net ~{MO3_0}: J1.28 (Pin_28), JP13.1 (A)
- new net ~{MO3_1}: J1.27 (Pin_27), JP14.1 (A)
- new net ~{MO3_2}: J1.26 (Pin_26), JP15.1 (A)
- new net ~{MO3_3}: J1.25 (Pin_25), JP16.1 (A)
- new net ~{MO_S0_0}: JP5.2 (C)
- new net ~{MO_S0_1}: JP6.2 (C)
- new net ~{MO_S0_2}: JP7.2 (C)
- new net ~{MO_S0_3}: JP8.2 (C)
- new net ~{MO_S1_0}: JP13.2 (C)
- new net ~{MO_S1_1}: JP14.2 (C)
- new net ~{MO_S1_2}: JP15.2 (C)
- new net ~{MO_S1_3}: JP16.2 (C)
- new net ~{RAM_CLK}: J1.21 (Pin_21), U3.11, U3.8
- new net ~{RAM_EN}: J1.22 (Pin_22), U4.32 (OE#), U6.32 (OE#)
- new net ~{ROM_EN}: J1.19 (Pin_19), U3.2, U3.5
- new net ~{SEL_0}: JP17.2 (C), U3.3, U3.9
- new net ~{SEL_1}: JP18.2 (C), U3.12, U3.6
Other:
- added sheet samp32-memory-mux (samp32-memory-mux.kicad_sch)
- added sheet samp32-memory-mux1 (samp32-memory-mux.kicad_sch)
- added sheet scamp32-memory-address-adder (scamp32-memory-address-adder.kicad_sch)
- added sheet scamp32-memory-data-bus (scamp32-memory-data-bus.kicad_sch)
- added sheet scamp32-memory-data-bus1 (scamp32-memory-data-bus.kicad_sch)
- note added: "For memory card 1, JP1: 2-3, JP2: 2-3 For memory card 2, JP1: 1-3, JP2: 1-3"
